File: hardware/android-box-rebuild/6_PERF1.kicad_sch (KiCad schematic)
At the start: 82 parts, among them U14 T527, U17 SY6280AAC

Commit message: Add J6 USB-C host schematic
Parts:
- USB2, USB3: now not fitted; now left out of the parts list
Changed lines of the file:
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@@
 		(body_style 0)
 		(exclude_from_sim no)
-		(in_bom yes)
-		(on_board yes)
-		(in_pos_files yes)
-		(dnp no)
+		(in_bom no)
+		(on_board no)
+		(in_pos_files no)
+		(dnp yes)
 		(property "Reference" "USB2"
 			(at 332.74 196.85 0)
@@
 		(body_style 0)
 		(exclude_from_sim no)
-		(in_bom yes)
-		(on_board yes)
-		(in_pos_files yes)
-		(dnp no)
+		(in_bom no)
+		(on_board no)
+		(in_pos_files no)
+		(dnp yes)
 		(property "Reference" "USB3"
 			(at 175.26 237.49 0)
