File: hardware/android-box-rebuild/android-box-rebuild.kicad_sch (KiCad schematic)
At the start: 0 parts

Commit message: Route J5 USB-C PD power front end
Other:
- added sheet USB-C PD 9V INPUT (USB_C_PD_9V.kicad_sch)
- sheet 12VDC ports: added PD_9V_PROTECTED; removed none
Changed lines of the file:
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@@
 	(generator_version "10.0")
 	(paper "A4")
+	(wire
+		(pts
+			(xy 17.78 104.775) (xy 45 104.775)
+		)
+		(stroke
+			(width 0)
+			(type default)
+		)
+	)
 	(sheet
 		(at 5.08 102.87)
@@
 			)
 		)
+		(pin "PD_9V_PROTECTED" input
+			(at 17.78 104.775 0)
+			(effects
+				(font
+					(size 1.27 1.27)
+				)
+				(justify right)
+			)
+		)
 		(instances
 			(project "avaota-a1-v14"
@@
 				)
 			)
+		)
+	)
+	(sheet
+		(at 45 102.87)
+		(size 35.56 3.81)
+		(exclude_from_sim no)
+		(in_bom yes)
+		(on_board yes)
+		(dnp no)
+		(fields_autoplaced yes)
+		(stroke
+			(width 0.1524)
+			(type solid)
+		)
+		(fill
+			(color 0 0 0 0)
+		)
+		(property "Sheetname" "USB-C PD 9V INPUT"
+			(at 45 102.1584 0)
+			(show_name no)
+			(do_not_autoplace no)
+			(effects
+				(font
+					(size 1.27 1.27)
+				)
+				(justify left bottom)
+			)
+		)
+		(property "Sheetfile" "USB_C_PD_9V.kicad_sch"
+			(at 45 107.2646 0)
+			(show_name no)
+			(do_not_autoplace no)
+			(effects
+				(font
+					(size 1.27 1.27)
+				)
+				(justify left top)
+			)
+		)
+		(pin "PD_9V_PROTECTED" output
+			(at 45 104.775 180)
+			(effects
+				(font
+					(size 1.27 1.27)
+				)
+				(justify left)
+			)
+		)
+		(instances
+			(project "avaota-a1-v14"
+				(path "/550d58f0-4e41-4062-aec4-b3409407efa1"
+					(page "15")
+				)
+			)

Commit message: Add J6 USB-C host schematic
Other:
- added sheet USB-C HOST J6 (USB_C_HOST.kicad_sch)
Changed lines of the file:
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@@
+		)
+	)
+	(sheet
+		(at 45 110.49)
+		(size 35.56 3.81)
+		(exclude_from_sim no)
+		(in_bom yes)
+		(on_board yes)
+		(dnp no)
+		(fields_autoplaced yes)
+		(stroke (width 0.1524) (type solid))
+		(fill (color 0 0 0 0))
+		(property "Sheetname" "USB-C HOST J6"
+			(at 45 109.7784 0)
+			(show_name no)
+			(do_not_autoplace no)
+			(effects (font (size 1.27 1.27)) (justify left bottom))
+		)
+		(property "Sheetfile" "USB_C_HOST.kicad_sch"
+			(at 45 114.8846 0)
+			(show_name no)
+			(do_not_autoplace no)
+			(effects (font (size 1.27 1.27)) (justify left top))
+		)
+		(instances
+			(project "avaota-a1-v14"
+				(path "/550d58f0-4e41-4062-aec4-b3409407efa1" (page "16"))
+			)
 		)
 	)
